File: 3-Phase_Motor_Driver.kicad_sch (KiCad schematic)
At the start: 26 parts, among them J1 Conn_01x05_Male, J2 USB4105-GF-A, SW1 Boot0, SW2 RESET, U1 DRV8323RSRGZR, U2 STM32G441KBT3

Commit message: Added more to schematic
Parts:
- removed C10: 1uF/16V, symbol Device:C
- removed C11, C7, C8, C9: 100nF/10V, symbol Device:C
- removed J1: Conn_01x05_Male, symbol Connector:Conn_01x05_Male
- removed R4, R5: R, symbol Device:R
- removed R6, R7: 10k/1%/0.1W, symbol Device:R
- removed SW1: Boot0, symbol Switch:SW_DIP_x01
- removed SW2: RESET, symbol Switch:SW_DIP_x01
- removed U2: STM32G441KBT3, LQFP32_7X7_STM, symbol STM32G441KBT:STM32G441KBT3
- added C12: 47nF/X7R/50V, Capacitor_SMD:C_0603_1608Metric, symbol Device:C
- added C13: 100nF/X7R/50V, Capacitor_SMD:C_0603_1608Metric, symbol Device:C
- added C14, C15, C16: 10uF/X7R/50V, Capacitor_SMD:C_1206_3216Metric, symbol Device:C
- added C17: 2.2uF/100V/X7R, Capacitor_SMD:C_1206_3216Metric, symbol Device:C
- added C18, C19: 1uF/16V, Capacitor_SMD:C_0603_1608Metric, symbol Device:C
- added J3: Conn_01x06_Male, ul_B6B-PH-K-S-LF-SN:B6B-PH-K-SLFSN, symbol Connector:Conn_01x06_Male
- added L2: 22uH/300mA, CBC2518T220M:INDC2518X200N, symbol Device:L
- added NT1: NetTie_2, symbol Device:NetTie_2
- added R8, R9: 10k/1%/0.1W, Resistor_SMD:R_0603_1608Metric, symbol Device:R
- added U3: LTC3631EMS8E-5-TRPBF, ul_LTC3631EMS8E-5-TRPBF:LTC3631EMS8E-5-TRPBF, symbol ul_LTC3631EMS8E-5-TRPBF:LTC3631EMS8E-5-TRPBF
- added U4: LP5907MFX-3.3/NOPB, LP5907MFX-3:SOT95P280X145-5N, symbol LP5907MFX-3.3_NOPB:LP5907MFX-3.3/NOPB
- C1, C2, C3, C5: footprint (none) -> Capacitor_SMD:C_0603_1608Metric
- C4: value 2.2uF/100V/10% -> 2.2uF/100V/X7R; footprint (none) -> Capacitor_SMD:C_1206_3216Metric
- C6: value 10uF/25V/10% -> 10uF/X7R/50V; footprint (none) -> Capacitor_SMD:C_1206_3216Metric; MPN GRM188R61E106KA73D -> CL31A106MBHNNNE; Supplier_PN 490-18214-1-ND -> 1276-6736-1-ND
- D1: footprint (none) -> Diode_SMD:D_SOD-128
- J2: footprint GCT_USB4105-GF-A -> USB4105-GF-A:GCT_USB4105-GF-A; Supplier (none) -> Digikey
- L1: footprint (none) -> ul_ASPI-0628-4R7M-T1:ASPI-0628-4R7M-T1
- R1, R2, R3: footprint (none) -> Resistor_SMD:R_0603_1608Metric
- U1: footprint QFN50P700X700X100-49N -> DRV8323RSRGZR:QFN50P700X700X100-49N
Connections:
- net +3.3VA: now also R8.1, R9.2
- net GND: now also U1.2 (PGND), U1.43 (BGND), C13.2, C14.2, C15.2, NT1.2; no longer J2.A1_B12 (GND), J2.B1_A12 (GND), J2.S1 (SHELL_GND), J2.S2 (SHELL_GND), J2.S3 (SHELL_GND), J2.S4 (SHELL_GND)
- net at J2.A4_B9 (VBUS), J2.B4_A9 (VBUS): now also C18.1, U4.1 (IN), U4.3 (EN)
- net GLA: now reaches U1.10 (GLA)
- net SPA: now reaches U1.11 (SPA)
- net SNA: now reaches U1.12 (SNA)
- net SNB: now reaches U1.13 (SNB)
- net SPB: now reaches U1.14 (SPB)
- net GLB: now reaches U1.15 (GLB)
- net SHB: now reaches U1.16 (SHB)
- net GHB: now reaches U1.17 (GHB)
- net GHC: now reaches U1.18 (GHC)
- net SHC: now reaches U1.19 (SHC)
- net GLC: now reaches U1.20 (GLC)
- net SPC: now reaches U1.21 (SPC)
- net SNC: now reaches U1.22 (SNC)
- net SOC: now reaches U1.23 (SOC)
- net SOB: now reaches U1.24 (SOB)
- net SOA: now reaches U1.25 (SOA)
- net GNDD: now reaches U1.27 (DGND)
- net GNDD: now also J2.A1_B12 (GND), J2.B1_A12 (GND), J2.S1 (SHELL_GND), J2.S2 (SHELL_GND), J2.S3 (SHELL_GND), J2.S4 (SHELL_GND), U1.35 (AGND), U1.49 (EP), C16.2, C17.2, C18.2, C19.2, J3.1 (Pin_1), NT1.1, U3.8 (GND), U4.2 (GND)
- net FAULT: now reaches U1.28 (FAULT_N)
- net FAULT: now also R8.2
- net MISO: now reaches U1.29 (SDO)
- net MISO: now also R9.1
- net at U1.3 (CPL): now also C12.2
- net MOSI: now reaches U1.30 (SDI)
- net SCK: now reaches U1.31 (SCLK)
- net CS: now reaches U1.32 (SCS_N)
- net ENABLE: now reaches U1.33 (ENABLE)
- net CAL: now reaches U1.34 (CAL)
- net at U1.4 (CPH): now also C12.1
- net GHA: now reaches U1.8 (GHA)
- net SHA: now reaches U1.9 (SHA)
- net Vbatt renamed VIN
- net VIN: now also C13.1, C14.1, C15.1, C17.1, U3.2 (VIN), U3.5 (RUN)
- new net: L2.2, U3.1 (SW)
- new net +3V3: C19.1, U4.5 (OUT)
- new net +5V: C16.1, J3.6 (Pin_6), L2.1, U3.6 (VOUT/VFB)
- new net HALL_A: J3.4 (Pin_4)
- new net HALL_B: J3.3 (Pin_3)
- new net HALL_C: J3.2 (Pin_2)
- new net TEMP: J3.5 (Pin_5)
- no-connect marks 2 -> 7
Other:
- added sheet Controller (Controller.kicad_sch)
- added sheet MOSFETS (MOSFETS.kicad_sch)
- note added: "ENCODER INPUT"
- note added: "Notes: Select current sense gain to be 20V/V Frequency is (TBD)"
- note added: "Tie this pin close to MOSFET section"
- note added: "USB INTERFACE"
- moved on the sheet: C1, C4, R1

Commit message: Updated Schematics and worked on board layout
Parts:
- removed U3: LTC3631EMS8E-5-TRPBF, ul_LTC3631EMS8E-5-TRPBF:LTC3631EMS8E-5-TRPBF, symbol ul_LTC3631EMS8E-5-TRPBF:LTC3631EMS8E-5-TRPBF
- removed U4: LP5907MFX-3.3/NOPB, LP5907MFX-3:SOT95P280X145-5N, symbol LP5907MFX-3.3_NOPB:LP5907MFX-3.3/NOPB
- added C20: C_Polarized, symbol Device:C_Polarized
- added C21: 10uF/X7R/63V, Capacitor_SMD:C_1210_3225Metric, symbol Device:C
- added H1, H2: MountingHole_Pad, MountingHole:MountingHole_2.7mm, symbol Mechanical:MountingHole_Pad
- added U3: FAN48610UC50X, ul_FAN48610UC50X:FAN48610UC50X, symbol ul_FAN48610UC50X:FAN48610UC50X
- added U4: LP5907MFX-3.3/NOPB, LP5907MFX-3:SOT95P280X145-5N, symbol LP5907MFX-3.3_NOPB:LP5907MFX-3.3_NOPB
- C13: value 100nF/X7R/50V -> 100nF/X7R/100V; MPN CL10B104KB8WPNC -> CL10B104KC8NNNC; Supplier_PN 1276-6854-1-ND -> 1276-6807-1-ND
- C14, C15, C16, C6: value 10uF/X7R/50V -> 10uF/X7R/63V; footprint Capacitor_SMD:C_1206_3216Metric -> Capacitor_SMD:C_1210_3225Metric; MPN CL31A106MBHNNNE -> CL32B106KMVNNWE; Supplier_PN 1276-6736-1-ND -> 1276-7053-1-ND
- L2: value 22uH/300mA -> 0.47uH/1A; footprint CBC2518T220M:INDC2518X200N -> Inductor_SMD:L_1008_2520Metric; MPN CBC2518T220M -> CIGT252010LMR47MNE; Supplier_PN 587-1616-1-ND -> 1276-6944-1-ND
- NT1: footprint (none) -> NetTie:NetTie-4_SMD_Pad2.0mm
Connections:
- net +3.3VA: now also C17.1, L2.1, U3.A3 (VIN), U3.B3 (EN)
- net +3V3: now also U4.5 (OUT)
- net +5V: now also U3.A1 (VOUT), U3.A2 (VOUT); no longer L2.1
- net GND: now also U1.49 (EP), C20.2, C21.2, H2.1
- net GNDD: now also U3.C1 (PGND), U3.C2 (PGND), U3.C3 (AGND), U4.2 (GND); no longer U1.49 (EP)
- net VIN: now also C20.1, C21.1, H1.1; no longer C17.1
- net at C18.1, J2.A4_B9 (VBUS), J2.B4_A9 (VBUS): now also U4.1 (IN), U4.3 (EN)
- net at L2.2: now also U3.B1 (SW), U3.B2 (SW)
- no-connect marks 7 -> 4
Other:
- note added: "Notes: Select current sense gain to be 20V/V Frequency is >30kHz"
- note added: "Place close to MOSFETS to reduce dV/dt"
- note removed: "Notes: Select current sense gain to be 20V/V Frequency is (TBD)"
- moved on the sheet: C16, C17, L2
