File: Controller.kicad_sch (KiCad schematic)
At the start: 13 parts, among them J1 Conn_02x05_Odd_Even, Q13 Q_PMOS_GDS, SW1 RESET, SW2 Boot0, U2 STM32G441KBT6

Commit message: Updated Schematics and worked on board layout
Parts:
- removed SW1: RESET, symbol Switch:SW_DIP_x01
- added SW1: EVQ-P7J01P, EVQ-P7J01P:SW_EVQ-P7J01P, symbol EVQ-P7J01P:EVQ-P7J01P
- C11, C7, C8, C9: value 100nF/X7R/50V -> 100nF/X7R/100V; MPN CL10B104KB8WPNC -> CL10B104KC8NNNC; Supplier_PN 1276-6854-1-ND -> 1276-6807-1-ND
- SW2: footprint (none) -> Connector_PinHeader_2.54mm:PinHeader_1x03_P2.54mm_Horizontal
Connections:
- net GNDD: now also SW1.2_1, SW1.2_2
- net NRST: now also SW1.1_1, SW1.1_2
- no-connect marks 0 -> 1
Other:
- moved on the sheet: C10, C7, C8, C9, U2B
